File: DCMv3/DCMv3.sch (EAGLE design)
At the start: 27 parts, among them IC1 OKI-78SR-5_1.5-W36H-C, J1 DT15-12PA, J2 DTM15-12PA, M1 DRV8872DDA, Q1 IPD50P04P4L-11, U1 A000005, U2 TLE94108EL

Commit message: updating DCMv3
x
Parts:
- removed U$2: SM6T39A, SM6T39A:SM6T39A
- removed U$3: 47UF, EEE-FC1C471AP:47UF
- added C5: EEE-FT1H470AP, SamacSys_Parts:EEE-FT1H470AP
- added Z1: MM3Z12VT1G, SamacSys_Parts:MM3Z12VT1G
- C1: value EEE-HDV470XAP -> EEE-FT1H470AP; device SamacSys_Parts:EEE-HDV470XAP -> SamacSys_Parts:EEE-FT1H470AP
- D1: value 1SMA5927BT3G -> SM6T39A; device 1sma59xx_10:1SMA5927BT3G -> SamacSys_Parts:SM6T39A
Connections:
- removed net MIR_SEL: R3.2, U1.A6_MIR_SEL
- removed net N$18: U1.A1
- removed net P_WIN: U1.A3_P_WIN
- new net N$6: J2.6
- new net N$7: J2.7
- net FOLD_A: now also J1.8
- net FOLD_B: now also J1.9
- net GATE: now also Z1.A; no longer D1.A
- net GND: now also C5.-, D1.A, J1.2, J1.3; no longer J1.6, U$2.A, U$3.-
- net ILLUM_IN: now also R3.2, U1.A6_MIR_SEL; no longer U1.A2_ILLUM_IN
- net IN1: now also U1.A2_ILLUM_IN
- net IN2: now also U1.A3_P_WIN
- net MIR_COM: now also J1.5
- net MIR_H: now also J1.4
- net MIR_V: now also J1.7
- net N$10: now also J2.10; no longer J1.10
- net N$13: now also J2.11; no longer J1.11
- net N$2: now also J2.2; no longer J1.2
- net N$3: now also J2.3; no longer J1.3
- net N$4: now also J2.4; no longer J1.4
- net N$5: now also J2.5; no longer J1.5
- net N$8: now also J2.8; no longer J1.8
- net N$9: now also J2.9; no longer J1.9
- net NFAULT: now also U1.A1
- net RX: now also J2.1
- net TX: now also J2.12
- net VBAT: now also J1.10, J1.11; no longer J1.7
- net VS: now also C5.+, D1.K, Z1.K; no longer D1.C, U$2.C, U$3.+
Other:
- moved on the sheet: C1, D1, R10

Commit message: added current sense resistor
Parts:
- removed R9: UCR006YVPFLR120, SamacSys_Parts:UCR006YVPFLR120
- added R1: RLP73K3AR12FTDF, SamacSys_Parts:RLP73K3AR12FTDF
Connections:
- net GND: now also R1.2; no longer R9.2
- net ISEN: now also R1.1; no longer R9.1
Changed lines of the file:
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@@
 <part name="R8" library="SamacSys_Parts" deviceset="ERJ-1RKD4700C" device=""/>
 <part name="GND6" library="supply1" library_urn="urn:adsk.eagle:library:371" deviceset="GND" device=""/>
-<part name="R9" library="SamacSys_Parts" deviceset="UCR006YVPFLR120" device=""/>
 <part name="C3" library="SamacSys_Parts" deviceset="GRM033R6YA104KE14D" device=""/>
 <part name="J2" library="DTM15-12PA" deviceset="DTM15-12PA" device=""/>
@@
 <part name="C5" library="SamacSys_Parts" deviceset="EEE-FT1H470AP" device=""/>
 <part name="GND2" library="supply1" library_urn="urn:adsk.eagle:library:371" deviceset="GND" device=""/>
+<part name="R1" library="SamacSys_Parts" deviceset="RLP73K3AR12FTDF" device=""/>
 </parts>
 <sheets>
@@
 <attribute name="VALUE" x="-33.02" y="129.54" size="1.778" layer="96"/>
 </instance>
-<instance part="R9" gate="G$1" x="15.24" y="66.04" smashed="yes">
-<attribute name="NAME" x="22.352" y="66.04" size="1.778" layer="95" align="center-left"/>
-</instance>
 <instance part="C3" gate="G$1" x="15.24" y="58.42" smashed="yes" rot="R270">
 <attribute name="NAME" x="11.43" y="52.07" size="1.778" layer="95" rot="R270" align="center-left"/>
@@
 <instance part="GND2" gate="1" x="25.4" y="40.64" smashed="yes">
 <attribute name="VALUE" x="22.86" y="38.1" size="1.778" layer="96"/>
+</instance>
+<instance part="R1" gate="G$1" x="15.24" y="66.04" smashed="yes">
+<attribute name="NAME" x="29.21" y="72.39" size="1.778" layer="95" align="center-left"/>
+<attribute name="VALUE" x="29.21" y="69.85" size="1.778" layer="96" align="center-left"/>
 </instance>
 </instances>
@@
 <pinref part="GND3" gate="1" pin="GND"/>
 <wire x1="43.18" y1="66.04" x2="43.18" y2="63.5" width="0.1524" layer="91"/>
-<pinref part="R9" gate="G$1" pin="2"/>
+<pinref part="R1" gate="G$1" pin="2"/>
 </segment>
 <segment>
@@
 <pinref part="M1" gate="G$1" pin="ISEN"/>
 <wire x1="7.62" y1="66.04" x2="15.24" y2="66.04" width="0.1524" layer="91"/>
-<pinref part="R9" gate="G$1" pin="1"/>
+<pinref part="R1" gate="G$1" pin="1"/>
 </segment>
 </net>

Commit message: WIP
Other:
- moved on the sheet: M1
